File: hardware/kicad/power_switch_and_regulator.kicad_sch (KiCad schematic)
At the start: 10 parts, among them Q5 PMV32UP, U4 XC6220, U5 TPL5110DDCR

Commit message: schematic restructure update
Connections:
- net BATT+ renamed +BATT
