File: hardware/kicad/solar_power.kicad_sch (KiCad schematic)
At the start: 12 parts, among them U4 AEM10941

Commit message: wip: revision 2
Connections:
- net MPP_STATUS: now reaches U4.19 (STATUS[2])
- no-connect marks 7 -> 6
Changed lines of the file:
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@@
   (no_connect (at 192.405 82.55))
   (no_connect (at 233.045 90.17))
-  (no_connect (at 233.045 102.87))
   (no_connect (at 233.045 92.71))
   (wire (pts (xy 179.705 100.33) (xy 189.865 100.33))
@@
     (stroke (width 0.5) (type default))
   )
+  (wire (pts (xy 233.045 102.87) (xy 240.03 102.87))
+    (stroke (width 0) (type default))
+  )
   (wire (pts (xy 192.405 105.41) (xy 189.865 105.41))
     (stroke (width 0) (type default))
@@
     (effects (font (size 1.27 1.27)) (justify left))
   )
+  (hierarchical_label "MPP_STATUS" (shape output) (at 240.03 102.87 0) (fields_autoplaced)
+    (effects (font (size 1.27 1.27)) (justify left))
+  )

Commit message: fix schematic info
Other:
- company: (none) -> Teapot Laboratories
- title: (none) -> Solar Power
Changed lines of the file:
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@@
   (paper "A4")
   (title_block
-    (date "2023-10-16")
-    (rev "2")
+    (title "Solar Power")
+    (date "2024-01-10")
+    (rev "3")
+    (company "Teapot Laboratories")
   )
   (junction (at 98.425 78.74) (diameter 0) (color 0 0 0 0)

Commit message: update bom
Parts:
- SC1: value KXOB25-05X3TF-TR -> KXOB25-05X3F-TR; Distributor Link https://www.digikey.com/en/products/detail/anysolar-ltd/KXOB25-05X3TF-TR/13999164 -> https://www.digikey.com/en/products/detail/anysolar-ltd/KXOB25-05X3F-TR/9990478; Distributor Part Number 2994-KXOB25-05X3TF-TRCT-ND -> KXOB25-05X3FCT-ND; Manufacturer Part Number KXOB25-05X3TF-TR -> KXOB25-05X3F-TR; Part Description Solar Cell G3 Thin 2.07V 30.9MW -> Solar Cell G3 Thin 2.07V 30.7MW
- SC2, SC3, SC4: renamed from SC1; value KXOB25-05X3TF-TR -> KXOB25-05X3F-TR; Distributor Link https://www.digikey.com/en/products/detail/anysolar-ltd/KXOB25-05X3TF-TR/13999164 -> https://www.digikey.com/en/products/detail/anysolar-ltd/KXOB25-05X3F-TR/9990478; Distributor Part Number 2994-KXOB25-05X3TF-TRCT-ND -> KXOB25-05X3FCT-ND; Manufacturer Part Number KXOB25-05X3TF-TR -> KXOB25-05X3F-TR; Part Description Solar Cell G3 Thin 2.07V 30.9MW -> Solar Cell G3 Thin 2.07V 30.7MW
- renumbered C14 to C21, C14 to C22, C17 to C23, L2 to L3, L3 to L4, TP4 to TP3, TP5 to TP4
