File: hardware/kicad/sensor.kicad_sch (KiCad schematic)
At the start: 20 parts, among them Q2 PMV32UP, Q3 DMG1012UW, Q6 MMBT3906, U2 BME688

Commit message: schematic restructure update
Parts:
- removed R13, R14: 10K, Resistor_SMD:R_0603_1608Metric, symbol Device:R_Small
Connections:
- net BATT+ renamed +BATT
Other:
- moved on the sheet: R11

Commit message: beautify schematic
Other:
- note added: "Environmental Sensor"
- note added: "Sheets Connection"
- note removed: "BME680 Environmental Sensor over I2C"
- moved on the sheet: C10, C19, C20, C30, D3, Q2, Q3, Q6, R11, R12, R19, R22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

Commit message: sensor sch partially done
Parts:
- removed C10: 0.1uF, Capacitor_SMD:C_0603_1608Metric, symbol Device:C
- removed C19, C20: 100nF, Capacitor_SMD:C_0603_1608Metric_Pad1.08x0.95mm_HandSolder, symbol Device:C_Small
- removed R11, R12: 10K, Resistor_SMD:R_0603_1608Metric_Pad0.98x0.95mm_HandSolder, symbol Device:R_Small
- removed R6: 10K, Resistor_SMD:R_0603_1608Metric, symbol Device:R_Small
- removed R7, R8: 1M, Resistor_SMD:R_0603_1608Metric, symbol Device:R_Small
- added C27 (x3): 100n, Capacitor_SMD:C_0402_1005Metric, symbol Device:C_Small
- added R13 (x3): 10K, Resistor_SMD:R_0603_1608Metric, symbol Device:R_Small
- added R16 (x2): 1M, Resistor_SMD:R_0603_1608Metric_Pad0.98x0.95mm_HandSolder, symbol Device:R_Small
- Q2: Distributor (none) -> LCSC; Distributor Link (none) -> https://www.lcsc.com/product-detail/MOSFETs_TECH-PUBLIC-PMV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; Distributor Part Number (none) -> C2959851; Manufacturer (none) -> TECH PUBLIC; Manufacturer Part Number (none) -> PMV32UP; Part Description (none) -> MOSFET P Channel 20V 4A 52mΩ@4.5V
- Q3: Distributor (none) -> LCSC; Distributor Link (none) -> https://www.lcsc.com/product-detail/MOSFETs_Diodes-Incorpor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; Distributor Part Number (none) -> C156390; Manufacturer (none) -> Diodes Incorporated; Manufacturer Part Number (none) -> DMG1012UW-7; Part Description (none) -> MOSFET N Channel 20V 1A 450mΩ@4.5V 600mA 290mW
- R5: value 4.7K -> 4K7; footprint Resistor_SMD:R_0603_1608Metric -> Resistor_SMD:R_0402_1005Metric; Distributor (none) -> LCSC; Distributor Link (none) -> https://www.lcsc.com/product-detail/Chip-Resistor-Surface-M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; Distributor Part Number (none) -> C25900; Manufacturer (none) -> UNI-ROYAL(Uniroyal Elec); Manufacturer Part Number (none) -> 0402WGF4701TCE; Part Description (none) -> Resistor 62.5mW ±1% 4.7kΩ
- U2: footprint Teapot:BME680-PSON80P300X300X100-8N -> plantpal:BME680-PSON80P300X300X100-8N; Distributor (none) -> LCSC; Distributor Link (none) -> https://www.digikey.com/en/products/detail/bosch-sensortec/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; Distributor Part Number (none) -> 828-BME688CT-ND; Manufacturer (none) -> Bosch Sensortec; Manufacturer Part Number (none) -> BME688; Part Description (none) -> Gas, Humidity, Pressure, Temperature Sensor I²C, SPI Output
Connections:
- net +3V3: now also C27.1, C27.2, R13.2, R13.2
- net +BATT: now also R16.1
- net BATT_MEAS: now also C27.1, R13.2
- net BATT_MEAS_EN: now also R16.1
- net GND: now also C27.1, C27.2, C27.2, R13.1, R16.2
- net at Q2.1 (G), Q3.3 (D): now also R16.2
- net at U2.5 (SDO): now also R13.1
- net at U2.2 (CSB): now also R13.1

Commit message: sensor sch done
Parts:
- removed R19, R24: 10k, Resistor_SMD:R_0402_1005Metric, symbol Device:R_Small_US
- removed R22: 1M, Resistor_SMD:R_0402_1005Metric, symbol Device:R_Small_US
- added R13 (x2): 10K, Resistor_SMD:R_0603_1608Metric, symbol Device:R_Small
- added R16: 1M, Resistor_SMD:R_0603_1608Metric_Pad0.98x0.95mm_HandSolder, symbol Device:R_Small
- C30: Distributor (none) -> LCSC; Distributor Link (none) -> https://www.lcsc.com/product-detail/Multilayer-Ceramic-Capa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; Distributor Part Number (none) -> C14442; LCSC C1523 -> (none); Manufacturer (none) -> Samsung Electro-Mechanics; Manufacturer Part Number (none) -> CL05B102KB5NNNC; Part Description (none) -> Ceramic Capacitors 50V 1nF X7R ±10%
- D3: Distributor (none) -> LCSC; Distributor Link (none) -> https://www.lcsc.com/product-detail/Switching-Diode_ST-Semt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; Distributor Part Number (none) -> C9808; LCSC C9808 -> (none); Manufacturer (none) -> ST(Semtech); Manufacturer Part Number (none) -> LL4148; Part Description (none) -> Switching Diode 75V 500mW 1V@10mA 4ns 0.2A
- Q6: Distributor (none) -> LCSC; Distributor Link (none) -> https://www.lcsc.com/product-detail/Bipolar-Transistors-BJT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; Distributor Part Number (none) -> C2143; LCSC C2910191 -> (none); Manufacturer (none) -> Jiangsu Changjing Electronics Technology Co., Ltd.; Manufacturer Part Number (none) -> MMBT3906 2A; Part Description (none) -> Bipolar Transistors 40V 200mW 100@10mA,1V 200mA PNP
Connections:
- net CAP_TRACK: now also R13.1
- net GND: now also R16.2
- net PWM: now also R13.2, R13.2
- net SENSE_OUT: now also R16.1
- net at Q6.1 (B): now also R13.1

Commit message: change resistor to 0402
Parts:
- R13: footprint Resistor_SMD:R_0603_1608Metric -> Resistor_SMD:R_0402_1005Metric
- R16: footprint Resistor_SMD:R_0603_1608Metric_Pad0.98x0.95mm_HandSolder -> Resistor_SMD:R_0402_1005Metric
Changed lines of the file:
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@@
       (effects (font (size 1.27 1.27)) (justify left))
     )
-    (property "Footprint" "Resistor_SMD:R_0603_1608Metric" (at 118.11 60.96 0)
+    (property "Footprint" "Resistor_SMD:R_0402_1005Metric" (at 118.11 60.96 0)
       (effects (font (size 1.27 1.27)) hide)
     )
@@
       (effects (font (size 1.27 1.27)) (justify left))
     )
-    (property "Footprint" "Resistor_SMD:R_0603_1608Metric" (at 163.195 46.99 0)
+    (property "Footprint" "Resistor_SMD:R_0402_1005Metric" (at 163.195 46.99 0)
       (effects (font (size 1.27 1.27)) hide)
     )
@@
       (effects (font (size 1.27 1.27)) (justify left))
     )
-    (property "Footprint" "Resistor_SMD:R_0603_1608Metric_Pad0.98x0.95mm_HandSolder" (at 188.595 106.045 0)
+    (property "Footprint" "Resistor_SMD:R_0402_1005Metric" (at 188.595 106.045 0)
       (effects (font (size 1.27 1.27)) hide)
     )
@@
       (effects (font (size 1.27 1.27)) (justify left))
     )
-    (property "Footprint" "Resistor_SMD:R_0603_1608Metric" (at 118.11 76.2 0)
+    (property "Footprint" "Resistor_SMD:R_0402_1005Metric" (at 118.11 76.2 0)
       (effects (font (size 1.27 1.27)) hide)
     )
@@
       (effects (font (size 1.27 1.27)) (justify left))
     )
-    (property "Footprint" "Resistor_SMD:R_0603_1608Metric" (at 163.195 64.77 0)
+    (property "Footprint" "Resistor_SMD:R_0402_1005Metric" (at 163.195 64.77 0)
       (effects (font (size 1.27 1.27)) hide)
     )
@@
       (effects (font (size 1.27 1.27)) (justify left))
     )
-    (property "Footprint" "Resistor_SMD:R_0603_1608Metric" (at 173.99 133.985 0)
+    (property "Footprint" "Resistor_SMD:R_0402_1005Metric" (at 173.99 133.985 0)
       (effects (font (size 1.27 1.27)) hide)
     )
@@
       (effects (font (size 1.27 1.27)) (justify left))
     )
-    (property "Footprint" "Resistor_SMD:R_0603_1608Metric_Pad0.98x0.95mm_HandSolder" (at 198.755 122.555 0)
+    (property "Footprint" "Resistor_SMD:R_0402_1005Metric" (at 198.755 122.555 0)
       (effects (font (size 1.27 1.27)) hide)
     )
@@
       (effects (font (size 1.27 1.27)) (justify left))
     )
-    (property "Footprint" "Resistor_SMD:R_0603_1608Metric_Pad0.98x0.95mm_HandSolder" (at 210.185 52.07 0)
-      (effects (font (size 1.27 1.27)) hide)
-    )
+    (property "Footprint" "Resistor_SMD:R_0402_1005Metric" (at 210.185 52.07 0)
+      (effects (font (size 1.27 1.27)) hide)
+    )

Commit message: clean-up
Parts:
- U2: Distributor LCSC -> Digikey
Changed lines of the file:
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@@
       (effects (font (size 1.27 1.27)) hide)
     )
-    (property "Distributor" "LCSC" (at 96.52 68.58 0)
+    (property "Distributor" "Digikey" (at 96.52 68.58 0)
       (effects (font (size 1.27 1.27)) hide)
     )
