File: hardware/kicad/sensor.kicad_sch (KiCad schematic)
At the start: 18 parts, among them Q2 PMV32UP, Q3 DMG1012UW, Q6 MMBT3906, U2 BME688

Commit message: fix schematic info
Other:
- company: (none) -> Teapot Laboratories
- title: (none) -> Sensor
Changed lines of the file:
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@@
   (paper "A4")
   (title_block
-    (date "2023-10-16")
-    (rev "2")
+    (title "Sensor")
+    (date "2024-01-10")
+    (rev "3")
+    (company "Teapot Laboratories")
   )
   (junction (at 156.845 46.99) (diameter 0) (color 0 0 0 0)

Commit message: update bom
Parts:
- renumbered C27 to C28, C27 to C29, Q6 to Q3, Q2 to Q4, Q3 to Q5, R13 to R16, R13 to R17, R13 to R18, R13 to R19, R5 to R20, R13 to R21, R16 to R22, R16 to R23, R16 to R24, U2 to U7
