File: hardware/kicad/power_gate_and_regulator.kicad_sch (KiCad schematic)
At the start: 10 parts, among them Q5 PMV32UP, U4 XC6220, U5 TPL5110DDCR

Commit message: beautify schematic
Other:
- note added: "Max 1000mA"
- note added: "Power Gate"
- note added: "Power Regulator"
- note added: "Sheets Connection"
- note added: "Use better LDO with lower Iq"
- note removed: "3.3V Regulator (Max 1000mA)"
- moved on the sheet: C21, C22, C23, D2, Q5, R15, R20, TP6, U4, U5

Commit message: power gate reg partially done
Parts:
- removed C21: 10u, Capacitor_SMD:C_0603_1608Metric_Pad1.08x0.95mm_HandSolder, symbol Device:C_Small
- removed C23: 100nF, Capacitor_SMD:C_0603_1608Metric, symbol Device:C_Small
- removed Q5: PMV32UP, Package_TO_SOT_SMD:SOT-23, symbol Simulation_SPICE:PMOS
- removed U5: TPL5110DDCR, Teapot:SOT95P280X110-6N, symbol cwlr1a:TPL5110DDCR
- added C27: 100n, Capacitor_SMD:C_0402_1005Metric, symbol Device:C_Small
- added C28: 10u, Capacitor_SMD:C_0603_1608Metric, symbol Device:C_Small
- added Q8: DMG3415U-7, Package_TO_SOT_SMD:SOT-23, symbol Device:Q_PMOS_GSD
- added U9: TPL5110, Package_TO_SOT_SMD:SOT-23-6, symbol Timer:TPL5110
- D2: Distributor (none) -> LCSC; Distributor Link (none) -> https://www.lcsc.com/product-detail/Schottky-Barrier-Diodes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; Distributor Part Number (none) -> C109213; Manufacturer (none) -> Shikues; Manufacturer Part Number (none) -> B5819W; Part Description 0.05mA@40V 0.58V@1A -> SBD 0.05mA@40V 0.58V@1A
- R15: Distributor (none) -> LCSC; Distributor Link (none) -> https://www.lcsc.com/product-detail/Chip-span-style-backgro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; Distributor Part Number (none) -> C163488; Manufacturer (none) -> YAGEO; Manufacturer Part Number (none) -> RC0402FR-0716K9L; Part Description (none) -> Resistor 62.5mW ±1% 16.9kΩ
- R20: Distributor (none) -> LCSC; Distributor Link (none) -> https://www.lcsc.com/product-detail/Chip-span-style-backgro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; Distributor Part Number (none) -> C25744; Manufacturer (none) -> UNI-ROYAL(Uniroyal Elec); Manufacturer Part Number (none) -> 0402WGF1002TCE; Part Description (none) -> Resistor 62.5mW ±1% 10kΩ
- U4: Distributor (none) -> Mouser; Distributor Link (none) -> https://www.mouser.com/ProductDetail/Torex-Semiconductor/XC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; Distributor Part Number (none) -> 865-XC6220B331MR-G; Manufacturer (none) -> Torex Semiconductor; Manufacturer Part Number (none) -> XC6220B331MR-G; Part Description (none) -> LDO Voltage Regulators 1A
Connections:
- net +BATT: now also C27.1, Q8.2 (S), U9.1 (VDD), U9.6 (EN/ONE_SHOT)
- net DONE: now also U9.4 (DONE)
- net DRV: now also Q8.1 (G), U9.5 (DRV)
- net GND: now also C27.2, C28.2, U9.2 (GND)
- net M_DRV: now also U9.3 (DELAY/M_DRV)
- net at U4.1 (VIN): now also C28.1, Q8.3 (D)
Other:
- moved on the sheet: D2, R15, R20

Commit message: power gate reg done
Parts:
- removed C22: 10u, Capacitor_SMD:C_0603_1608Metric_Pad1.08x0.95mm_HandSolder, symbol Device:C_Small
- added C28: 10u, Capacitor_SMD:C_0603_1608Metric, symbol Device:C_Small
Connections:
- net +3V3: now also C28.1
- net GND: now also C28.2
Changed lines of the file:
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@@
-    )
-  )
-  (symbol (lib_id "Device:C_Small") (at 236.855 96.52 0) (unit 1)
-    (in_bom yes) (on_board yes) (dnp no)
-    (property "Reference" "C22" (at 242.57 96.52 0)
-      (effects (font (size 1.27 1.27)) (justify right))
-    )
-    (property "Value" "10u" (at 243.205 99.06 0)
-      (effects (font (size 1.27 1.27)) (justify right))
-    )
-    (property "Footprint" "Capacitor_SMD:C_0603_1608Metric_Pad1.08x0.95mm_HandSolder" (at 236.855 96.52 0)
-      (effects (font (size 1.27 1.27)) hide)
-    )
-    (property "Datasheet" "https://product.tdk.com/system/files/dam/doc/product/capacitor/ceramic/mlcc/catalog/mlcc_commercial_general_en.pdf" (at 236.855 96.52 0)
-      (effects (font (size 1.27 1.27)) hide)
-    )
-    (property "Mouser" "https://www.mouser.com/ProductDetail/Murata-Electronics/GRM188R61A226ME15D?qs=eeBpzGFlv%252B8DV%2FrilzyhAw%3D%3D&gclid=Cj0KCQjwn4qWBhCvARIsAFNAMijttFPRtrXWYJjjdc3F7Yr8ZlLfo9gaIVHNlfh9bZOT-ul2jVOpdVYaAk1sEALw_wcB" (at 236.855 96.52 0)
-      (effects (font (size 1.27 1.27)) hide)
-    )
-    (pin "1")
-    (pin "2")
-    (instances
-      (project "plantpal"
-        (path "/59b4123e-c7be-466b-a5db-658b8f0c1171"
-          (reference "C22") (unit 1)
-        )
-        (path "/59b4123e-c7be-466b-a5db-658b8f0c1171/0bc89df9-c404-42cc-aab4-4237df7294d4"
-          (reference "C26") (unit 1)
-        )
-      )
-      (project "bwlr1e"
-        (path "/630c8da6-5464-4eef-824d-89618087f4b4"
-          (reference "C14") (unit 1)
-        )
-      )
     )
   )
@@
         )
       )
+    )
+  )
+  (symbol (lib_id "Device:C_Small") (at 236.855 96.52 0) (mirror y) (unit 1)
+    (in_bom yes) (on_board yes) (dnp no)
+    (property "Reference" "C28" (at 234.315 95.2562 0)
+      (effects (font (size 1.27 1.27)) (justify left))
+    )
+    (property "Value" "10u" (at 234.315 97.7962 0)
+      (effects (font (size 1.27 1.27)) (justify left))
+    )
+    (property "Footprint" "Capacitor_SMD:C_0603_1608Metric" (at 236.855 96.52 0)
+      (effects (font (size 1.27 1.27)) hide)
+    )
+    (property "Datasheet" "https://datasheet.lcsc.com/lcsc/2304140030_Samsung-Electro-Mechanics-CL10A106KP8NNNC_C19702.pdf" (at 236.855 96.52 0)
+      (effects (font (size 1.27 1.27)) hide)
+    )
+    (property "Part Description" "Ceramic Capacitor 10V 10uF X5R ±10% 0603" (at 236.855 96.52 0)
+      (effects (font (size 1.27 1.27)) hide)
+    )
+    (property "Manufacturer" "Samsung Electro-Mechanics" (at 236.855 96.52 0)
+      (effects (font (size 1.27 1.27)) hide)
+    )
+    (property "Manufacturer Part Number" "CL10A106KP8NNNC" (at 236.855 96.52 0)
+      (effects (font (size 1.27 1.27)) hide)
+    )
+    (property "Distributor" "LCSC" (at 236.855 96.52 0)
+      (effects (font (size 1.27 1.27)) hide)
+    )
+    (property "Distributor Part Number" "C19702" (at 236.855 96.52 0)
+      (effects (font (size 1.27 1.27)) hide)
+    )
+    (property "Distributor Link" "https://www.lcsc.com/product-detail/Multilayer-Ceramic-Capacitors-MLCC-SMD-SMT_Samsung-Electro-Mechanics-CL10A106KP8NNNC_C19702.html" (at 236.855 96.52 0)
+      (effects (font (size 1.27 1.27)) hide)
+    )
+    (pin "1")
+    (pin "2")
+    (instances
+      (project "plantpal"
+        (path "/59b4123e-c7be-466b-a5db-658b8f0c1171"
+          (reference "C28") (unit 1)
+        )
+        (path "/59b4123e-c7be-466b-a5db-658b8f0c1171/7fda2409-1758-4461-822b-801ba75fe202"
+          (reference "C19") (unit 1)
+        )
+        (path "/59b4123e-c7be-466b-a5db-658b8f0c1171/0bc89df9-c404-42cc-aab4-4237df7294d4"
+          (reference "C26") (unit 1)
+        )
+      )
+      (project "bwlr1e-prog"
+        (path "/630c8da6-5464-4eef-824d-89618087f4b4"
+          (reference "C3") (unit 1)
+        )
+      )
+      (project "feather_rak3172"
+        (path "/a1545928-1195-40b9-b3c4-78f837012afb"
+          (reference "C6") (unit 1)
+        )
+      )

Commit message: clean-up
Parts:
- C27: Distributor Link https://www.lcsc.com/product-detail/Multilayer-Ceramic-Capacitors-MLCC-SMD-SMT_YAGEO-CC0402KRX5R6BB104_C129131.html -> https://www.lcsc.com/product-detail/Multilayer-Ceramic-Capacitors-MLCC-SMD-SMT_Samsung-Electro-Mechanics-CL05B104KO5NNNC_C1525.html; Distributor Part Number C129131 -> C1525; Manufacturer YAGEO -> Samsung Electro-Mechanics; Manufacturer Part Number CC0402KRX5R6BB104 -> CL05B104KO5NNNC; Part Description Ceramic Capacitor 10V 100nF X5R ±10% 0402 -> Ceramic Capacitor 16V 100nF X7R ±10%
- Q2: renamed from Q8; Part Description P Channel MOSFET 20V 4A 39mΩ@4.5V 4A 900mW -> MOSFET P Channel 20V 4A 39mΩ@4.5V 4A 900mW
- R15: value 16.9K -> 16K9
- renumbered U9 to U5

Commit message: clean-up
Parts:
- TP6: footprint TestPoint:TestPoint_Pad_D1.5mm -> TestPoint:TestPoint_Pad_D1.0mm
Changed lines of the file:
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@@
       (effects (font (size 1.27 1.27)))
     )
-    (property "Footprint" "TestPoint:TestPoint_Pad_D1.5mm" (at 237.49 64.135 0)
+    (property "Footprint" "TestPoint:TestPoint_Pad_D1.0mm" (at 237.49 64.135 0)
       (effects (font (size 1.27 1.27)) hide)
     )
@@
       (effects (font (size 1.27 1.27)) hide)
     )
+    (property "Part Description" "" (at 237.49 69.215 0)
+      (effects (font (size 1.27 1.27)) hide)
+    )
+    (property "Manufacturer" "" (at 237.49 69.215 0)
+      (effects (font (size 1.27 1.27)) hide)
+    )
+    (property "Manufacturer Part Number" "" (at 237.49 69.215 0)
+      (effects (font (size 1.27 1.27)) hide)
+    )
+    (property "Distributor" "" (at 237.49 69.215 0)
+      (effects (font (size 1.27 1.27)) hide)
+    )
+    (property "Distributor Part Number" "" (at 237.49 69.215 0)
+      (effects (font (size 1.27 1.27)) hide)
+    )
+    (property "Distributor Link" "" (at 237.49 69.215 0)
+      (effects (font (size 1.27 1.27)) hide)
+    )

Commit message: wip wake-up button
Parts:
- added Q2: PMV32UP, Package_TO_SOT_SMD:SOT-23, symbol Device:Q_PMOS_GSD
- added R17: 5K1, Resistor_SMD:R_0402_1005Metric, symbol Device:R_Small
Connections:
- net +BATT: now also Q2.2 (S)
- net M_DRV: now also R17.1
- new net: Q2.3 (D), R17.2
- new net CHIP_EN: Q2.1 (G)
Other:
- note added: "TODO: Fix CHIP_EN is floating when power is off"
- note added: "Wake-up Button"
