File: hardware/kicad/power_gate_and_regulator.kicad_sch (KiCad schematic)
At the start: 12 parts, among them Q2 DMG3415U-7, Q2 PMV32UP, U4 XC6220, U5 TPL5110

Commit message: wip wake-up button
Parts:
- added R16: 1M, Resistor_SMD:R_0402_1005Metric, symbol Device:R_Small
Connections:
- net +BATT: now also R16.2
- net CHIP_EN renamed RESET_BTN
- net RESET_BTN: now also R16.1
Other:
- note added: "TODO: verify if this circuit works"
- note removed: "TODO: Fix CHIP_EN is floating when power is off"
- moved on the sheet: Q2, R17

Commit message: wip wake up button
Other:
- note added: "TODO: make sure signal from +BATT to M_DRV never exceed 3V3"
- note added: "TODO: make sure signal from VBUS never exceed 3V3"
Changed lines of the file:
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@@
+    (effects (font (size 1.27 1.27)) (justify left bottom))
+  )
+  (text "TODO: make sure signal from +BATT to M_DRV never exceed 3V3"
+    (at 52.07 120.65 0)
     (effects (font (size 1.27 1.27)) (justify left bottom))
   )
@@
     (effects (font (size 1.27 1.27)) (justify left bottom))
   )
+  (text "TODO: make sure signal from VBUS never exceed 3V3" (at 50.165 112.395 0)
+    (effects (font (size 1 1)) (justify left bottom))
+  )
   (text "Wake-up\nButton" (at 52.705 130.81 0)

Commit message: wip wake up button
Other:
- note added: "TODO: make sure signal from VBUS to M_DRV never exceed 3V3"
- note added: "TODO: restructure schematic for M_DRV signaling"
- note removed: "TODO: make sure signal from VBUS never exceed 3V3"
Changed lines of the file:
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@@
     (effects (font (size 1.27 1.27)) (justify left bottom))
+  )
+  (text "TODO: restructure schematic for M_DRV signaling" (at 50.165 109.855 0)
+    (effects (font (size 1 1)) (justify left bottom))
   )
   (text "TODO: make sure signal from +BATT to M_DRV never exceed 3V3"
@@
     (effects (font (size 1.27 1.27)) (justify left bottom))
   )
-  (text "TODO: make sure signal from VBUS never exceed 3V3" (at 50.165 112.395 0)
+  (text "TODO: make sure signal from VBUS to M_DRV never exceed 3V3"
+    (at 50.165 112.395 0)
     (effects (font (size 1 1)) (justify left bottom))
   )

Commit message: wip wake up button
Parts:
- removed R17: 5K1, Resistor_SMD:R_0402_1005Metric, symbol Device:R_Small
- added R15: 16K9, Resistor_SMD:R_0402_1005Metric, symbol Device:R_Small
- Q2: value PMV32UP -> PMZ350UPEYL; footprint Package_TO_SOT_SMD:SOT-23 -> Package_TO_SOT_SMD:SOT-883; Distributor Link https://www.lcsc.com/product-detail/MOSFETs_TECH-PUBLIC-PMV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 -> https://www.lcsc.com/product-detail/MOSFETs_Nexperia-PMZ350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; Distributor Part Number C2959851 -> C478207; Manufacturer TECH PUBLIC -> Nexperia; Manufacturer Part Number PMV32UP -> PMZ350UPEYL; Part Description MOSFET P Channel 20V 4A 52mΩ@4.5V -> MOSFET P Channel 20V 1A 450mΩ@4.5V,300mA 360mW
Connections:
- net M_DRV: now also R20.1, R15.2; no longer R20.2
- net at D2.1 (K): now also R15.1; no longer R20.1
- net at Q2.3 (D): now also R20.2

Commit message: wip wake-up button
Other:
- note removed: "TODO: make sure signal from +BATT to M_DRV never exceed 3V3"
- note removed: "TODO: make sure signal from VBUS to M_DRV never exceed 3V3"
Changed lines of the file:
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@@
     (effects (font (size 1.27 1.27)) (justify left bottom))
   )
-  (text "TODO: restructure schematic for M_DRV signaling" (at 50.165 109.855 0)
+  (text "TODO: restructure schematic for M_DRV signaling" (at 49.53 112.395 0)
     (effects (font (size 1 1)) (justify left bottom))
-  )
-  (text "TODO: make sure signal from +BATT to M_DRV never exceed 3V3"
-    (at 52.07 120.65 0)
-    (effects (font (size 1.27 1.27)) (justify left bottom))
   )
   (text "Around 30s Timer" (at 84.455 97.155 0)
     (effects (font (size 1.27 1.27)) (justify left bottom))
   )
-  (text "TODO: make sure signal from VBUS to M_DRV never exceed 3V3"
-    (at 50.165 112.395 0)
-    (effects (font (size 1 1)) (justify left bottom))
-  )
   (text "Wake-up\nButton" (at 52.705 130.81 0)

Commit message: update library
Parts:
- Q2: footprint Package_TO_SOT_SMD:SOT-883 -> plantpal:SOT-883
Changed lines of the file:
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@@
       (effects (font (size 1.27 1.27)) (justify left))
     )
-    (property "Footprint" "Package_TO_SOT_SMD:SOT-883" (at 78.105 139.065 0)
+    (property "Footprint" "plantpal:SOT-883" (at 78.105 139.065 0)
       (effects (font (size 1.27 1.27)) hide)
     )
