File: hardware/kicad/power_gate_and_regulator.kicad_sch (KiCad schematic)
At the start: 13 parts, among them Q2 DMG3415U-7, Q2 PMZ350UPEYL, U4 XC6220, U5 TPL5110

Commit message: update bom
Parts:
- U4: Distributor Mouser -> LCSC; Distributor Link https://www.mouser.com/ProductDetail/Torex-Semiconductor/XC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 -> https://www.lcsc.com/product-detail/Linear-Voltage-Regulato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; Distributor Part Number 865-XC6220B331MR-G -> C86534
Changed lines of the file:
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@@
       (effects (font (size 1.27 1.27)) hide)
     )
-    (property "Distributor" "Mouser" (at 217.17 83.185 0)
+    (property "Distributor" "LCSC" (at 217.17 83.185 0)
       (effects (font (size 1.27 1.27)) hide)
     )
-    (property "Distributor Part Number" "865-XC6220B331MR-G" (at 217.17 83.185 0)
+    (property "Distributor Part Number" "C86534" (at 217.17 83.185 0)
       (effects (font (size 1.27 1.27)) hide)
     )
-    (property "Distributor Link" "https://www.mouser.com/ProductDetail/Torex-Semiconductor/XC6220B331MR-G?qs=AsjdqWjXhJ8lRh0WBUyqoQ%3D%3D" (at 217.17 83.185 0)
+    (property "Distributor Link" "https://www.lcsc.com/product-detail/Linear-Voltage-Regulators-LDO_Torex-Semicon-XC6220B331MR-G_C86534.html" (at 217.17 83.185 0)
       (effects (font (size 1.27 1.27)) hide)
     )
