File: hardware/kicad/plantpal.kicad_sch (KiCad schematic)
At the start: 0 parts

Commit message: work in progress
Other:
- sheet Display ports: added none; removed TSCL, TSDA
Changed lines of the file:
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@@
-    (stroke (width 0) (type default))
-  )
-  (wire (pts (xy 233.045 121.92) (xy 238.76 121.92))
     (stroke (width 0) (type default))
   )
@@
   )
   (wire (pts (xy 146.05 77.47) (xy 149.225 77.47))
-    (stroke (width 0) (type default))
-  )
-  (wire (pts (xy 233.045 119.38) (xy 238.76 119.38))
     (stroke (width 0) (type default))
   )
@@
   (wire (pts (xy 82.55 118.11) (xy 158.75 118.11))
     (stroke (width 0) (type default))
-  )
-  (label "SDA" (at 238.76 119.38 180) (fields_autoplaced)
-    (effects (font (size 1.27 1.27)) (justify right bottom))
-  )
-  (label "SCL" (at 238.76 121.92 180) (fields_autoplaced)
-    (effects (font (size 1.27 1.27)) (justify right bottom))
   )
   (label "SDA" (at 198.12 78.105 0) (fields_autoplaced)
@@
       (effects (font (size 1.27 1.27)) (justify left))
     )
-    (pin "TSDA" bidirectional (at 233.045 119.38 0)
-      (effects (font (size 1.27 1.27)) (justify right))
-    )
-    (pin "TSCL" input (at 233.045 121.92 0)
-      (effects (font (size 1.27 1.27)) (justify right))
-    )
     (pin "BUSY" output (at 214.63 109.22 180)

Commit message: wip wake-up button
Other:
- sheet Main Controller ports: added CHIP_EN; removed none
- sheet Power Gate and Regulator ports: added CHIP_EN; removed none
Changed lines of the file:
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@@
+    (stroke (width 0) (type default))
+  )
+  (wire (pts (xy 146.05 82.55) (xy 158.75 82.55))
     (stroke (width 0) (type default))
   )
@@
       (effects (font (size 1.27 1.27)) (justify right))
     )
+    (pin "CHIP_EN" input (at 146.05 82.55 0)
+      (effects (font (size 1.27 1.27)) (justify right))
+    )
     (instances
       (project "plantpal"
@@
       (effects (font (size 1.27 1.27)) (justify right))
     )
-    (instances
+    (pin "CHIP_EN" output (at 158.75 82.55 180)
+      (effects (font (size 1.27 1.27)) (justify left))
+    )
+    (instances

Commit message: wip wake-up button
Other:
- sheet Main Controller ports: added RESET_BTN; removed CHIP_EN
- sheet Power Gate and Regulator ports: added RESET_BTN; removed CHIP_EN
Changed lines of the file:
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@@
       (effects (font (size 1.27 1.27)) (justify right))
     )
-    (pin "CHIP_EN" input (at 146.05 82.55 0)
+    (pin "RESET_BTN" input (at 146.05 82.55 0)
       (effects (font (size 1.27 1.27)) (justify right))
     )
@@
       (effects (font (size 1.27 1.27)) (justify right))
     )
-    (pin "CHIP_EN" output (at 158.75 82.55 180)
-      (effects (font (size 1.27 1.27)) (justify left))
-    )
+    (pin "RESET_BTN" output (at 158.75 82.55 180)
+      (effects (font (size 1.27 1.27)) (justify left))
+    )

Commit message: wip wake up button
Changed lines of the file:
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@@
       (effects (font (size 1.27 1.27)) (justify left top))
-    )
-    (pin "M_DRV" bidirectional (at 146.05 87.63 0)
-      (effects (font (size 1.27 1.27)) (justify right))
     )
     (pin "DONE" input (at 146.05 85.09 0)
@@
       (effects (font (size 1.27 1.27)) (justify right))
     )
+    (pin "M_DRV" input (at 146.05 87.63 0)
+      (effects (font (size 1.27 1.27)) (justify right))
+    )
     (instances
       (project "plantpal"
@@
       (effects (font (size 1.27 1.27)) (justify right))
     )
-    (pin "M_DRV" bidirectional (at 158.75 87.63 180)
-      (effects (font (size 1.27 1.27)) (justify left))
-    )
     (pin "DONE" output (at 158.75 85.09 180)
       (effects (font (size 1.27 1.27)) (justify left))
@@
       (effects (font (size 1.27 1.27)) (justify left))
     )
+    (pin "M_DRV" output (at 158.75 87.63 180)
+      (effects (font (size 1.27 1.27)) (justify left))
+    )
