File: hardware/kicad/plantpal.kicad_pcb (KiCad board)
At the start: 2 copper layers, 38.4 x 128.5 mm, 120 parts, among them J1 U262-161N-4BVC11, J2 +LIPO, J3 -LIPO, J4 687124182122, Q1 DMG1012UW, Q2 DMG3415U-7, Q3 MMBT3906, Q4 PMV32UP, Q5 DMG1012UW, Q6 AO3407A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

Commit message: wip wake-up button
Parts:
- added D8: B5819W, Diode_SMD:D_SOD-123, F.Cu at (139.8, 48.1)
- added R28: 1M, Resistor_SMD:R_0402_1005Metric, F.Cu at (138.3, 52.8)
- moved Q8 150.1 mm to (142.7, 54.0)
- moved R27 146.4 mm to (137.4, 57.8)
Connections:
- Q8 pad 1: /Main Controller/CHIP_EN -> /Main Controller/RESET_BTN
- Q8 pad 3: (no net) -> Net-(Q8-D)
- R27 pad 1: Net-(Q8-D) -> /Main Controller/M_DRV
- R27 pad 2: /Main Controller/M_DRV -> Net-(Q8-D)
- SW2 pad 1: /Main Controller/CHIP_EN -> /Main Controller/RESET_BTN
Changed lines of the file:
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@@
   (net 88 "unconnected-(J4-TSDA-Pad7)")
   (net 89 "Net-(Q8-D)")
+  (net 90 "/Main Controller/RESET_BTN")
   (footprint "Capacitor_SMD:C_0402_1005Metric" (layer "F.Cu")
     (at 123.378 39.837)
@@
   )
   (footprint "Package_TO_SOT_SMD:SOT-23" (layer "F.Cu")
-    (at 1.945 1.725)
+    (at 142.7025 53.97)
     (descr "SOT, 3 Pin (https://www.jedec.org/system/files/docs/to-236h.pdf variant AB), generated with kicad-footprint-generator ipc_gullwing_generator.py")
     (tags "SOT TO_SOT_SMD")
@@
       (stroke (width 0.1) (type solid)) (layer "F.Fab"))
     (pad "1" smd roundrect (at -0.9375 -0.95) (size 1.475 0.6) (layers "F.Cu" "F.Paste" "F.Mask") (roundrect_rratio 0.25)
-      (net 11 "/Main Controller/CHIP_EN") (pinfunction "G") (pintype "input"))
+      (net 90 "/Main Controller/RESET_BTN") (pinfunction "G") (pintype "input"))
     (pad "2" smd roundrect (at -0.9375 0.95) (size 1.475 0.6) (layers "F.Cu" "F.Paste" "F.Mask") (roundrect_rratio 0.25)
       (net 16 "+BATT") (pinfunction "S") (pintype "passive"))
     (pad "3" smd roundrect (at 0.9375 0) (size 1.475 0.6) (layers "F.Cu" "F.Paste" "F.Mask") (roundrect_rratio 0.25)
-      (pinfunction "D") (pintype "passive"))
+      (net 89 "Net-(Q8-D)") (pinfunction "D") (pintype "passive"))
     (model "${KICAD6_3DMODEL_DIR}/Package_TO_SOT_SMD.3dshapes/SOT-23.wrl"
       (offset (xyz 0 0 0))
@@
     )
   )
+  (footprint "Diode_SMD:D_SOD-123" (layer "F.Cu")
+    (at 139.755 48.09)
+    (descr "SOD-123")
+    (tags "SOD-123")
+    (property "Distributor" "LCSC")
+    (property "Distributor Link" "https://www.lcsc.com/product-detail/Schottky-Barrier-Diodes-SBD_Shikues-B5819W_C109213.html")
+    (property "Distributor Part Number" "C109213")
+    (property "Manufacturer" "Shikues")
+    (property "Manufacturer Part Number" "B5819W")
+    (property "Part Description" "SBD 0.05mA@40V 0.58V@1A")
+    (property "Sheetfile" "main_controller.kicad_sch")
+    (property "Sheetname" "Main Controller")
+    (property "ki_description" "40V 0.5A Schottky Power Rectifier Diode, SOD-123")
+    (property "ki_keywords" "diode Schottky")
+    (attr smd)
+    (fp_text reference "D8" (at 0 -2) (layer "F.SilkS")
+        (effects (font (size 1 1) (thickness 0.15)))
+    )
+    (fp_text value "B5819W" (at 0 2.1) (layer "F.Fab")
+        (effects (font (size 1 1) (thickness 0.15)))
+    )
+    (fp_text user "${REFERENCE}" (at 0 -2) (layer "F.Fab")
+        (effects (font (size 1 1) (thickness 0.15)))
+    )
+    (fp_line (start -2.36 -1) (end -2.36 1)
+      (stroke (width 0.12) (type solid)) (layer "F.SilkS"))
+    (fp_line (start -2.36 -1) (end 1.65 -1)
+      (stroke (width 0.12) (type solid)) (layer "F.SilkS"))
+    (fp_line (start -2.36 1) (end 1.65 1)
+      (stroke (width 0.12) (type solid)) (layer "F.SilkS"))
+    (fp_line (start -2.35 -1.15) (end -2.35 1.15)
+      (stroke (width 0.05) (type solid)) (layer "F.CrtYd"))
+    (fp_line (start -2.35 -1.15) (end 2.35 -1.15)
+      (stroke (width 0.05) (type solid)) (layer "F.CrtYd"))
+    (fp_line (start 2.35 -1.15) (end 2.35 1.15)
+      (stroke (width 0.05) (type solid)) (layer "F.CrtYd"))
+    (fp_line (start 2.35 1.15) (end -2.35 1.15)
+      (stroke (width 0.05) (type solid)) (layer "F.CrtYd"))
+    (fp_line (start -1.4 -0.9) (end 1.4 -0.9)
+      (stroke (width 0.1) (type solid)) (layer "F.Fab"))
+    (fp_line (start -1.4 0.9) (end -1.4 -0.9)
+      (stroke (width 0.1) (type solid)) (layer "F.Fab"))
+    (fp_line (start -0.75 0) (end -0.35 0)
+      (stroke (width 0.1) (type solid)) (layer "F.Fab"))
+    (fp_line (start -0.35 0) (end -0.35 -0.55)
+      (stroke (width 0.1) (type solid)) (layer "F.Fab"))
+    (fp_line (start -0.35 0) (end -0.35 0.55)
+      (stroke (width 0.1) (type solid)) (layer "F.Fab"))
+    (fp_line (start -0.35 0) (end 0.25 -0.4)
+      (stroke (width 0.1) (type solid)) (layer "F.Fab"))
+    (fp_line (start 0.25 -0.4) (end 0.25 0.4)
+      (stroke (width 0.1) (type solid)) (layer "F.Fab"))
+    (fp_line (start 0.25 0) (end 0.75 0)
+      (stroke (width 0.1) (type solid)) (layer "F.Fab"))
+    (fp_line (start 0.25 0.4) (end -0.35 0)
+      (stroke (width 0.1) (type solid)) (layer "F.Fab"))
+    (fp_line (start 1.4 -0.9) (end 1.4 0.9)
+      (stroke (width 0.1) (type solid)) (layer "F.Fab"))
+    (fp_line (start 1.4 0.9) (end -1.4 0.9)
+      (stroke (width 0.1) (type solid)) (layer "F.Fab"))
+    (pad "1" smd roundrect (at -1.65 0) (size 0.9 1.2) (layers "F.Cu" "F.Paste" "F.Mask") (roundrect_rratio 0.25)
+      (net 90 "/Main Controller/RESET_BTN") (pinfunction "K") (pintype "passive"))
+    (pad "2" smd roundrect (at 1.65 0) (size 0.9 1.2) (layers "F.Cu" "F.Paste" "F.Mask") (roundrect_rratio 0.25)
+      (net 11 "/Main Controller/CHIP_EN") (pinfunction "A") (pintype "passive"))
+    (model "${KICAD6_3DMODEL_DIR}/Diode_SMD.3dshapes/D_SOD-123.wrl"
+      (offset (xyz 0 0 0))
+      (scale (xyz 1 1 1))
+      (rotate (xyz 0 0 0))
+    )
+  )
   (footprint "Package_DFN_QFN:QFN-28-1EP_5x5mm_P0.5mm_EP3.35x3.35mm" (layer "F.Cu")
     (at 106.71 57.01)
@@
   )
   (footprint "Resistor_SMD:R_0402_1005Metric" (layer "F.Cu")
-    (at 0.955 4.945)
+    (at 137.44 57.83)
     (descr "Resistor SMD 0402 (1005 Metric), square (rectangular) end terminal, IPC_7351 nominal, (Body size source: IPC-SM-782 page 72, https://www.pcb-3d.com/wordpress/wp-content/uploads/ipc-sm-782a_amendment_1_and_2.pdf), generated with kicad-footprint-generator")
     (tags "resistor")
@@
       (stroke (width 0.1) (type solid)) (layer "F.Fab"))
     (pad "1" smd roundrect (at -0.51 0) (size 0.54 0.64) (layers "F.Cu" "F.Paste" "F.Mask") (roundrect_rratio 0.25)
-      (net 89 "Net-(Q8-D)") (pintype "passive"))
-    (pad "2" smd roundrect (at 0.51 0) (size 0.54 0.64) (layers "F.Cu" "F.Paste" "F.Mask") (roundrect_rratio 0.25)
       (net 70 "/Main Controller/M_DRV") (pintype "passive"))
+    (pad "2" smd roundrect (at 0.51 0) (size 0.54 0.64) (layers "F.Cu" "F.Paste" "F.Mask") (roundrect_rratio 0.25)
+      (net 89 "Net-(Q8-D)") (pintype "passive"))
     (model "${KICAD6_3DMODEL_DIR}/Resistor_SMD.3dshapes/R_0402_1005Metric.wrl"
       (offset (xyz 0 0 0))
@@
     )
   )
+  (footprint "Resistor_SMD:R_0402_1005Metric" (layer "F.Cu")
+    (at 138.29 52.76)
+    (descr "Resistor SMD 0402 (1005 Metric), square (rectangular) end terminal, IPC_7351 nominal, (Body size source: IPC-SM-782 page 72, https://www.pcb-3d.com/wordpress/wp-content/uploads/ipc-sm-782a_amendment_1_and_2.pdf), generated with kicad-footprint-generator")
+    (tags "resistor")
+    (property "Distributor" "LCSC")
+    (property "Distributor Link" "https://www.lcsc.com/product-detail/Chip-Resistor-Surface-Mount_UNI-ROYAL-Uniroyal-Elec-0402WGF1004TCE_C26083.html")
+    (property "Distributor Part Number" "C26083")
+    (property "Manufacturer" "UNI-ROYAL(Uniroyal Elec)")
+    (property "Manufacturer Part Number" "0402WGF1004TCE")
+    (property "Part Description" "Resistor 62.5mW ±1% 1MΩ")
+    (property "Sheetfile" "power_gate_and_regulator.kicad_sch")
+    (property "Sheetname" "Power Gate and Regulator")
+    (property "ki_description" "Resistor, small symbol")
+    (property "ki_keywords" "R resistor")
+    (attr smd)
+    (fp_text reference "R28" (at 0 -1.17) (layer "F.SilkS")
+        (effects (font (size 1 1) (thickness 0.15)))
+    )
+    (fp_text value "1M" (at 0 1.17) (layer "F.Fab")
+        (effects (font (size 1 1) (thickness 0.15)))
+    )
+    (fp_text user "${REFERENCE}" (at 0 0) (layer "F.Fab")
+        (effects (font (size 0.26 0.26) (thickness 0.04)))
+    )
+    (fp_line (start -0.153641 -0.38) (end 0.153641 -0.38)
+      (stroke (width 0.12) (type solid)) (layer "F.SilkS"))
+    (fp_line (start -0.153641 0.38) (end 0.153641 0.38)
+      (stroke (width 0.12) (type solid)) (layer "F.SilkS"))
+    (fp_line (start -0.93 -0.47) (end 0.93 -0.47)
+      (stroke (width 0.05) (type solid)) (layer "F.CrtYd"))
+    (fp_line (start -0.93 0.47) (end -0.93 -0.47)
+      (stroke (width 0.05) (type solid)) (layer "F.CrtYd"))
+    (fp_line (start 0.93 -0.47) (end 0.93 0.47)
+      (stroke (width 0.05) (type solid)) (layer "F.CrtYd"))
+    (fp_line (start 0.93 0.47) (end -0.93 0.47)
+      (stroke (width 0.05) (type solid)) (layer "F.CrtYd"))
+    (fp_line (start -0.525 -0.27) (end 0.525 -0.27)
+      (stroke (width 0.1) (type solid)) (layer "F.Fab"))
+    (fp_line (start -0.525 0.27) (end -0.525 -0.27)
+      (stroke (width 0.1) (type solid)) (layer "F.Fab"))
+    (fp_line (start 0.525 -0.27) (end 0.525 0.27)
+      (stroke (width 0.1) (type solid)) (layer "F.Fab"))
+    (fp_line (start 0.525 0.27) (end -0.525 0.27)
+      (stroke (width 0.1) (type solid)) (layer "F.Fab"))
+    (pad "1" smd roundrect (at -0.51 0) (size 0.54 0.64) (layers "F.Cu" "F.Paste" "F.Mask") (roundrect_rratio 0.25)
+      (net 90 "/Main Controller/RESET_BTN") (pintype "passive"))
+    (pad "2" smd roundrect (at 0.51 0) (size 0.54 0.64) (layers "F.Cu" "F.Paste" "F.Mask") (roundrect_rratio 0.25)
+      (net 16 "+BATT") (pintype "passive"))
+    (model "${KICAD6_3DMODEL_DIR}/Resistor_SMD.3dshapes/R_0402_1005Metric.wrl"
+      (offset (xyz 0 0 0))
+      (scale (xyz 1 1 1))
+      (rotate (xyz 0 0 0))
+    )
+  )
   (footprint "Inductor_SMD:L_0402_1005Metric" (layer "F.Cu")
     (at 119.215 38.696 -90)
@@
       (stroke (width 0.1) (type solid)) (layer "F.Fab"))
     (pad "1" smd rect (at -1.7 0 270) (size 0.9 1.7) (layers "F.Cu" "F.Paste" "F.Mask")
-      (net 11 "/Main Controller/CHIP_EN") (pinfunction "1") (pintype "passive"))
+      (net 90 "/Main Controller/RESET_BTN") (pinfunction "1") (pintype "passive"))
     (pad "2" smd rect (at 1.7 0 270) (size 0.9 1.7) (layers "F.Cu" "F.Paste" "F.Mask")
       (net 2 "GND") (pinfunction "2") (pintype "passive"))

Commit message: wip
Parts:
- added D7: RB161QS-40T18R, Diode_SMD:D_0402_1005Metric, F.Cu at (109.8, 47.6)
- D8: value B5819W -> RB161QS-40T18R; footprint Diode_SMD:D_SOD-123 -> Diode_SMD:D_0402_1005Metric
- Q8: value PMV32UP -> PMZ350UPEYL; footprint Package_TO_SOT_SMD:SOT-23 -> Package_TO_SOT_SMD:SOT-883
- R14: value 10K -> 16K9
- R27: value 5K1 -> 10K
- moved Q8 25.3 mm to (117.5, 56.2), turned to 180 degrees
- moved R27 20.0 mm to (117.4, 57.4), turned to 180 degrees
- moved R28 19.7 mm to (118.9, 56.5), turned to 90 degrees
- moved D8 17.8 mm to (125.8, 37.1), turned to 180 degrees
- moved D3 0.54 mm to (125.6, 52.7)
- moved C13 0.54 mm to (125.8, 42.8)
- moved C30 0.54 mm to (123.4, 50.1)
- moved Q3 0.54 mm to (126.3, 49.9)
- moved R24 0.54 mm to (123.4, 51.0)
- moved SW1 0.54 mm to (126.5, 45.7)
- moved SW2 0.54 mm to (126.5, 40.0)
- moved R8 0.54 mm to (127.6, 42.8)
- moved Q5 0.06 mm to (95.6, 59.0)
Connections:
- TP9 pad 1: /Main Controller/CHIP_EN -> /Main Controller/RESET_BTN
- U1 pad 10: /Main Controller/M_DRV -> /Main Controller/M_DRVOUT
Routing:
- net /Main Controller/RESET_BTN: track 0.00 -> 44.9 mm, vias 0 -> 3
- net /Main Controller/CHIP_EN: track 47.6 -> 18.3 mm, vias 3 -> 2
- net /Main Controller/M_DRVOUT: track 0.00 -> 9.33 mm, vias 0 -> 2
- net +BATT: track 39.2 -> 47.4 mm
- net /Main Controller/M_DRV: track 13.4 -> 21.1 mm
- net /Main Controller/BOOT_MODE1: track 25.5 -> 22.7 mm
- net GND: track 18.9 -> 21.0 mm, vias 184 -> 186
- net /Main Controller/PWR_STATUS: track 10.1 -> 8.65 mm
- net Net-(Q8-D): track 0.00 -> 1.33 mm
- net /Sensor/CAP_TRACK: track 125.3 -> 124.7 mm
- net Net-(Q3-B): track 1.56 -> 2.18 mm
- net /Main Controller/SENSE_OUT: track 8.52 -> 9.14 mm

Commit message: wip
Routing:
- net GND: vias 186 -> 188
Changed lines of the file:
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@@
   (via (at 125.85 33.79) (size 0.6) (drill 0.3) (layers "F.Cu" "B.Cu") (free) (net 2))
   (via (at 97.17 34.37) (size 0.6) (drill 0.3) (layers "F.Cu" "B.Cu") (free) (net 2))
+  (via (at 122.01 38.65) (size 0.6) (drill 0.3) (layers "F.Cu" "B.Cu") (free) (net 2))
   (via (at 123.06 64.94) (size 0.6) (drill 0.3) (layers "F.Cu" "B.Cu") (free) (net 2))
   (via (at 121.64 65.02) (size 0.6) (drill 0.3) (layers "F.Cu" "B.Cu") (free) (net 2))
@@
   (via (at 116.24 67.72) (size 0.6) (drill 0.3) (layers "F.Cu" "B.Cu") (free) (net 2))
   (via (at 127.61 48.8) (size 0.6) (drill 0.3) (layers "F.Cu" "B.Cu") (free) (net 2))
+  (via (at 125.16 43.69) (size 0.6) (drill 0.3) (layers "F.Cu" "B.Cu") (free) (net 2))
   (via (at 106.72 56.96) (size 0.6) (drill 0.3) (layers "F.Cu" "B.Cu") (net 2))
   (via (at 120.07 43.12) (size 0.6) (drill 0.3) (layers "F.Cu" "B.Cu") (net 2))
