File: hardware/kicad/usb_power.kicad_sch (KiCad schematic)
At the start: 14 parts, among them J1 U262-161N-4BVC11, U6 USBLC6-2P6, U7 MCP73831T-2ACI/OT

Commit message: change usb polarity
Connections:
- net D_IN+: now also U6.3 (I/O2); no longer U6.1 (I/O1)
- net D_IN-: now also U6.1 (I/O1); no longer U6.3 (I/O2)
- net USB_D+: now also U6.4 (I/O2); no longer U6.6 (I/O1)
- net USB_D-: now also U6.6 (I/O1); no longer U6.4 (I/O2)
Changed lines of the file:
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@@
     (stroke (width 0) (type default))
   )
-  (wire (pts (xy 56.515 68.58) (xy 64.77 68.58))
+  (wire (pts (xy 93.345 68.58) (xy 85.09 68.58))
     (stroke (width 0) (type default))
   )
@@
     (stroke (width 0.5) (type default))
   )
-  (wire (pts (xy 85.09 68.58) (xy 93.345 68.58))
+  (wire (pts (xy 64.77 68.58) (xy 56.515 68.58))
     (stroke (width 0) (type default))
   )
@@
     (effects (font (size 1.27 1.27)) (justify right bottom))
   )
-  (label "D_IN-" (at 93.345 68.58 180) (fields_autoplaced)
+  (label "D_IN-" (at 56.515 68.58 0) (fields_autoplaced)
+    (effects (font (size 1.27 1.27)) (justify left bottom))
+  )
+  (label "D_IN+" (at 93.345 68.58 180) (fields_autoplaced)
     (effects (font (size 1.27 1.27)) (justify right bottom))
   )
-  (label "D_IN+" (at 56.515 68.58 0) (fields_autoplaced)
-    (effects (font (size 1.27 1.27)) (justify left bottom))
-  )
-  (hierarchical_label "USB_D-" (shape output) (at 87.63 63.5 0) (fields_autoplaced)
-    (effects (font (size 1.27 1.27)) (justify left))
+  (hierarchical_label "USB_D-" (shape output) (at 62.23 63.5 180) (fields_autoplaced)
+    (effects (font (size 1.27 1.27)) (justify right))
   )
   (hierarchical_label "+BATT" (shape bidirectional) (at 185.42 78.74 0) (fields_autoplaced)
@@
     (effects (font (size 1.27 1.27)) (justify right))
   )
-  (hierarchical_label "USB_D+" (shape output) (at 62.23 63.5 180) (fields_autoplaced)
-    (effects (font (size 1.27 1.27)) (justify right))
+  (hierarchical_label "USB_D+" (shape output) (at 87.63 63.5 0) (fields_autoplaced)
+    (effects (font (size 1.27 1.27)) (justify left))
   )
   (symbol (lib_id "Device:Polyfuse") (at 98.425 30.48 90) (unit 1)

Commit message: add testpad and wip
Parts:
- added TP3: VBUS_IN, TestPoint:TestPoint_Pad_D1.0mm, symbol Connector:TestPoint
Connections:
- net at C12.1, FB1.1, J1.A4 (VBUS)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: now also TP3.1
Changed lines of the file:
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@@
   (junction (at 80.01 30.48) (diameter 0) (color 0 0 0 0)
+  )
+  (junction (at 54.61 30.48) (diameter 0) (color 0 0 0 0)
   )
   (no_connect (at 45.72 60.96))
@@
     (stroke (width 0) (type default))
   )
+  (wire (pts (xy 54.61 27.305) (xy 54.61 30.48))
+    (stroke (width 0) (type default))
+  )
   (polyline (pts (xy 113.03 68.58) (xy 113.03 19.05))
     (stroke (width 0.5) (type default))
   )
-  (wire (pts (xy 45.72 30.48) (xy 80.01 30.48))
+  (wire (pts (xy 45.72 30.48) (xy 54.61 30.48))
     (stroke (width 0) (type default))
   )
@@
   )
   (wire (pts (xy 184.15 76.2) (xy 184.15 78.74))
+    (stroke (width 0) (type default))
+  )
+  (wire (pts (xy 54.61 30.48) (xy 80.01 30.48))
     (stroke (width 0) (type default))
   )
@@
         )
       )
+    )
+  )
+  (symbol (lib_id "Connector:TestPoint") (at 54.61 27.305 0) (unit 1)
+    (in_bom yes) (on_board yes) (dnp no)
+    (property "Reference" "TP3" (at 49.53 24.13 0)
+      (effects (font (size 1.27 1.27)) (justify left))
+    )
+    (property "Value" "VBUS_IN" (at 55.88 24.13 0)
+      (effects (font (size 1.27 1.27)) (justify left))
+    )
+    (property "Footprint" "TestPoint:TestPoint_Pad_D1.0mm" (at 59.69 27.305 0)
+      (effects (font (size 1.27 1.27)) hide)
+    )
+    (property "Datasheet" "~" (at 59.69 27.305 0)
+      (effects (font (size 1.27 1.27)) hide)
+    )
+    (property "Part Description" "" (at 54.61 27.305 0)
+      (effects (font (size 1.27 1.27)) hide)
+    )
+    (property "Manufacturer" "" (at 54.61 27.305 0)
+      (effects (font (size 1.27 1.27)) hide)
+    )
+    (property "Manufacturer Part Number" "" (at 54.61 27.305 0)
+      (effects (font (size 1.27 1.27)) hide)
+    )
+    (property "Distributor" "" (at 54.61 27.305 0)
+      (effects (font (size 1.27 1.27)) hide)
+    )
+    (property "Distributor Part Number" "" (at 54.61 27.305 0)
+      (effects (font (size 1.27 1.27)) hide)
+    )
+    (property "Distributor Link" "" (at 54.61 27.305 0)
+      (effects (font (size 1.27 1.27)) hide)
+    )
+    (pin "1")
+    (instances
+      (project "plantpal"
+        (path "/59b4123e-c7be-466b-a5db-658b8f0c1171"
+          (reference "TP3") (unit 1)
+        )
+        (path "/59b4123e-c7be-466b-a5db-658b8f0c1171/943ab7c0-d00c-4ea0-8716-990ca6b0cb6f"
+          (reference "TP7") (unit 1)
+        )
+        (path "/59b4123e-c7be-466b-a5db-658b8f0c1171/7fda2409-1758-4461-822b-801ba75fe202"
+          (reference "TP8") (unit 1)
+        )
+      )

Commit message: change charge rate to 1A
Parts:
- R21: value 2K -> 1K; Distributor Link https://www.lcsc.com/product-detail/Chip-span-style-backgro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 -> https://www.lcsc.com/product-detail/Chip-Resistor-Surface-M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; Distributor Part Number C4109 -> C11702; Manufacturer Part Number 0402WGF2001TCE -> 0402WGF1001TCE; Part Description Resistor 62.5mW ±1% 2kΩ -> Resistor 62.5mW ±1% 1kΩ
Other:
- note added: "Charge Rate: 1000mA"
- note removed: "Charge Rate: 500mA"
Changed lines of the file:
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@@
     (effects (font (size 1.27 1.27) (thickness 0.6) bold) (justify left bottom))
   )
-  (text "Charge Rate: 500mA" (at 124.46 33.02 0)
+  (text "Charge Rate: 1000mA" (at 124.46 33.02 0)
     (effects (font (size 1.27 1.27)) (justify left bottom))
   )
@@
       (effects (font (size 1.27 1.27)) (justify left))
     )
-    (property "Value" "2K" (at 135.89 40.64 90)
+    (property "Value" "1K" (at 135.89 40.64 90)
       (effects (font (size 1.27 1.27)) (justify left))
     )
@@
       (effects (font (size 1.27 1.27)) hide)
     )
-    (property "Datasheet" "https://datasheet.lcsc.com/lcsc/2206010230_UNI-ROYAL-Uniroyal-Elec-0402WGF2001TCE_C4109.pdf" (at 135.255 43.18 0)
-      (effects (font (size 1.27 1.27)) hide)
-    )
-    (property "Part Description" "Resistor 62.5mW ±1% 2kΩ " (at 135.255 43.18 0)
+    (property "Datasheet" "https://datasheet.lcsc.com/lcsc/2206010216_UNI-ROYAL-Uniroyal-Elec-0402WGF1001TCE_C11702.pdf" (at 135.255 43.18 0)
+      (effects (font (size 1.27 1.27)) hide)
+    )
+    (property "Part Description" "Resistor 62.5mW ±1% 1kΩ " (at 135.255 43.18 0)
       (effects (font (size 1.27 1.27)) hide)
     )
@@
       (effects (font (size 1.27 1.27)) hide)
     )
-    (property "Manufacturer Part Number" "0402WGF2001TCE" (at 135.255 43.18 0)
+    (property "Manufacturer Part Number" "0402WGF1001TCE" (at 135.255 43.18 0)
       (effects (font (size 1.27 1.27)) hide)
     )
@@
       (effects (font (size 1.27 1.27)) hide)
     )
-    (property "Distributor Part Number" "C4109" (at 135.255 43.18 0)
-      (effects (font (size 1.27 1.27)) hide)
-    )
-    (property "Distributor Link" "https://www.lcsc.com/product-detail/Chip-span-style-background-color-ff0-Resistor-span-Surface-Mount_UNI-ROYAL-Uniroyal-Elec-0402WGF2001TCE_C4109.html" (at 135.255 43.18 0)
-      (effects (font (size 1.27 1.27)) hide)
-    )
+    (property "Distributor Part Number" "C11702" (at 135.255 43.18 0)
+      (effects (font (size 1.27 1.27)) hide)
+    )
+    (property "Distributor Link" "https://www.lcsc.com/product-detail/Chip-Resistor-Surface-Mount_UNI-ROYAL-Uniroyal-Elec-0402WGF1001TCE_C11702.html" (at 135.255 43.18 0)
+      (effects (font (size 1.27 1.27)) hide)
+    )

Commit message: update bom
Parts:
- U7: Distributor Mouser -> LCSC; Distributor Link https://www.mouser.com/ProductDetail/Microchip-Technology/M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 -> https://www.lcsc.com/product-detail/Battery-Management-ICs_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; Distributor Part Number 579-MCP73831T-2ACIOT -> C424093; Manufacturer Microchip Technology -> Microchip Tech
Changed lines of the file:
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@@
       (effects (font (size 1.27 1.27)) hide)
     )
-    (property "Manufacturer" "Microchip Technology" (at 150.495 40.64 0)
+    (property "Manufacturer" "Microchip Tech" (at 150.495 40.64 0)
       (effects (font (size 1.27 1.27)) hide)
     )
@@
       (effects (font (size 1.27 1.27)) hide)
     )
-    (property "Distributor" "Mouser" (at 150.495 40.64 0)
+    (property "Distributor" "LCSC" (at 150.495 40.64 0)
       (effects (font (size 1.27 1.27)) hide)
     )
-    (property "Distributor Part Number" "579-MCP73831T-2ACIOT" (at 150.495 40.64 0)
+    (property "Distributor Part Number" "C424093" (at 150.495 40.64 0)
       (effects (font (size 1.27 1.27)) hide)
     )
-    (property "Distributor Link" "https://www.mouser.com/ProductDetail/Microchip-Technology/MCP73831T-2ACI-OT?qs=yUQqVecv4qvbBQBGbHx0Mw%3D%3D" (at 150.495 40.64 0)
+    (property "Distributor Link" "https://www.lcsc.com/product-detail/Battery-Management-ICs_Microchip-Tech-MCP73831T-2ACI-OT_C424093.html" (at 150.495 40.64 0)
       (effects (font (size 1.27 1.27)) hide)
     )

Commit message: hardware/kicad/battery.kicad_sch
Other:
- note added: "USB trace is less than Critical Length (2.4 inch) for USB2.0 Full-speed specification. No need for impedance control."
Changed lines of the file:
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@@
 (kicad_sch (version 20230121) (generator eeschema)
   (paper "A5")
+  (title_block
+    (date "2023-10-16")
+    (rev "2")
+  )
   (junction (at 92.71 30.48) (diameter 0) (color 0 0 0 0)
   )
@@
     (effects (font (size 1.27 1.27)) (justify left bottom))
   )
+  (text "USB trace is less than \nCritical Length (2.4 inch) for\nUSB2.0 Full-speed specification.\n\nNo need for impedance control."
+    (at 83.82 85.09 0)
+    (effects (font (size 1 1)) (justify left bottom))
+  )
   (label "D_IN-" (at 52.07 45.72 180) (fields_autoplaced)

Commit message: update incorrect D1 value
Parts:
- D1: value VLMO1500-GS08 -> VLMO1300-GS08; Distributor Link https://www.lcsc.com/product-detail/Light-Emitting-Diodes-s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 -> https://www.lcsc.com/product-detail/Light-Emitting-Diodes-L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; Distributor Part Number C3000857 -> C5184984; Manufacturer Part Number VLMO1500-GS08 -> VLMO1300-GS08
Changed lines of the file:
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@@
       (effects (font (size 1.27 1.27)))
     )
-    (property "Value" "VLMO1500-GS08" (at 178.435 36.83 0)
+    (property "Value" "VLMO1300-GS08" (at 178.435 36.83 0)
       (effects (font (size 1.27 1.27)))
     )
@@
       (effects (font (size 1.27 1.27)) hide)
     )
-    (property "Datasheet" "https://datasheet.lcsc.com/lcsc/2205051716_Vishay-Intertech-VLMO1500-GS08_C3000857.pdf" (at 174.625 36.195 0)
+    (property "Datasheet" "https://datasheet.lcsc.com/lcsc/2209291030_Vishay-Intertech-VLMO1300-GS08_C5184984.pdf" (at 174.625 36.195 0)
       (effects (font (size 1.27 1.27)) hide)
     )
@@
       (effects (font (size 1.27 1.27)) hide)
     )
-    (property "Manufacturer Part Number" "VLMO1500-GS08" (at 174.625 36.195 0)
+    (property "Manufacturer Part Number" "VLMO1300-GS08" (at 174.625 36.195 0)
       (effects (font (size 1.27 1.27)) hide)
     )
@@
       (effects (font (size 1.27 1.27)) hide)
     )
-    (property "Distributor Part Number" "C3000857" (at 174.625 36.195 0)
+    (property "Distributor Part Number" "C5184984" (at 174.625 36.195 0)
       (effects (font (size 1.27 1.27)) hide)
     )
-    (property "Distributor Link" "https://www.lcsc.com/product-detail/Light-Emitting-Diodes-span-style-background-color-ff0-LED-span_Vishay-Intertech-VLMO1500-GS08_C3000857.html" (at 174.625 36.195 0)
+    (property "Distributor Link" "https://www.lcsc.com/product-detail/Light-Emitting-Diodes-LED_Vishay-Intertech-VLMO1300-GS08_C5184984.html" (at 174.625 36.195 0)
       (effects (font (size 1.27 1.27)) hide)
     )

Commit message: wip
Parts:
- FB1: symbol Penguino-STM32WL-LoRa-E5-rescue:Ferrite_Bead-Device -> Device:FerriteBead
Changed lines of the file:
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@@
     )
   )
-  (symbol (lib_id "Penguino-STM32WL-LoRa-E5-rescue:Ferrite_Bead-Device") (at 87.63 30.48 90) (unit 1)
+  (symbol (lib_id "Device:FerriteBead") (at 87.63 30.48 90) (unit 1)
     (in_bom yes) (on_board yes) (dnp no)
     (property "Reference" "FB1" (at 84.455 29.21 90)
@@
       (effects (font (size 1.27 1.27)) hide)
     )
-    (property "Datasheet" "https://datasheet.lcsc.com/lcsc/2304140030_TDK-MMZ1608B601CTAH0_C97120.pdf" (at 87.63 30.48 0)
+    (property "Datasheet" "~" (at 87.63 30.48 0)
       (effects (font (size 1.27 1.27)) hide)
     )

Commit message: revision 3 prod
Changed lines of the file:
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@@
     (stroke (width 0) (type default))
   )
-  (polyline (pts (xy 165.1 69.85) (xy 165.1 86.36))
+  (polyline (pts (xy 174.625 69.85) (xy 174.625 86.36))
     (stroke (width 0) (type dash))
   )
@@
     (stroke (width 0) (type default))
   )
-  (polyline (pts (xy 195.58 69.85) (xy 165.1 69.85))
+  (polyline (pts (xy 195.58 69.85) (xy 174.625 69.85))
     (stroke (width 0) (type dash))
   )
@@
     (stroke (width 0.5) (type default))
   )
-  (wire (pts (xy 177.8 78.74) (xy 177.8 76.2))
-    (stroke (width 0) (type default))
-  )
   (polyline (pts (xy 111.125 93.98) (xy 111.125 19.05))
     (stroke (width 0.5) (type default))
@@
     (stroke (width 0) (type default))
   )
-  (wire (pts (xy 175.26 78.74) (xy 177.8 78.74))
-    (stroke (width 0) (type default))
-  )
   (wire (pts (xy 69.85 35.56) (xy 69.85 39.37))
     (stroke (width 0) (type default))
@@
     (stroke (width 0.5) (type default))
   )
-  (polyline (pts (xy 165.1 86.36) (xy 195.58 86.36))
+  (polyline (pts (xy 174.625 86.36) (xy 195.58 86.36))
     (stroke (width 0) (type dash))
   )
@@
   (hierarchical_label "+BATT" (shape bidirectional) (at 185.42 78.74 0) (fields_autoplaced)
     (effects (font (size 1.27 1.27)) (justify left))
-  )
-  (hierarchical_label "VBUS" (shape output) (at 175.26 78.74 180) (fields_autoplaced)
-    (effects (font (size 1.27 1.27)) (justify right))
   )
   (hierarchical_label "USB_D+" (shape output) (at 87.63 63.5 0) (fields_autoplaced)
@@
       (effects (font (size 1.27 1.27)) hide)
     )
-    (property "Datasheet" "~" (at 87.63 30.48 0)
+    (property "Datasheet" "https://datasheet.lcsc.com/lcsc/2304140030_TDK-MMZ1608B601CTAH0_C97120.pdf" (at 87.63 30.48 0)
       (effects (font (size 1.27 1.27)) hide)
     )
@@
         )
       )
-    )
-  )
-  (symbol (lib_id "power:VBUS") (at 177.8 76.2 0) (unit 1)
-    (in_bom yes) (on_board yes) (dnp no)
-    (property "Reference" "#PWR060" (at 177.8 80.01 0)
-      (effects (font (size 1.27 1.27)) hide)
-    )
-    (property "Value" "VBUS" (at 177.8 72.39 0)
-      (effects (font (size 1.27 1.27)))
-    )
-    (property "Footprint" "" (at 177.8 76.2 0)
-      (effects (font (size 1.27 1.27)) hide)
-    )
-    (property "Datasheet" "" (at 177.8 76.2 0)
-      (effects (font (size 1.27 1.27)) hide)
-    )
-    (pin "1")
-    (instances
-      (project "plantpal"
-        (path "/59b4123e-c7be-466b-a5db-658b8f0c1171"
-          (reference "#PWR060") (unit 1)
-        )
-        (path "/59b4123e-c7be-466b-a5db-658b8f0c1171/7fda2409-1758-4461-822b-801ba75fe202"
-          (reference "#PWR045") (unit 1)
-        )
-      )
-      (project "bwlr1e-prog"
-        (path "/630c8da6-5464-4eef-824d-89618087f4b4"
-          (reference "#PWR014") (unit 1)
-        )
-      )
-      (project "Penguino-STM32WL-LoRa-E5"
-        (path "/c338af29-f8d9-4513-836a-55ed8bfc47d3"
-          (reference "#PWR0105") (unit 1)
-        )
-      )
