File: hardware/kicad/usb_power.kicad_sch (KiCad schematic)
At the start: 15 parts, among them J1 U262-161N-4BVC11, U6 USBLC6-2P6, U7 MCP73831T-2ACI/OT

Commit message: fix schematic info
Other:
- company: (none) -> Teapot Laboratories
- title: (none) -> USB Power
Changed lines of the file:
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@@
   (paper "A5")
   (title_block
-    (date "2023-10-16")
-    (rev "2")
+    (title "USB Power")
+    (date "2024-01-10")
+    (rev "3")
+    (company "Teapot Laboratories")
   )
   (junction (at 92.71 30.48) (diameter 0) (color 0 0 0 0)

Commit message: update bom
Parts:
- R12: renamed from R21; value 1K -> 2K; Distributor Link https://www.lcsc.com/product-detail/Chip-Resistor-Surface-Mount_UNI-ROYAL-Uniroyal-Elec-0402WGF1001TCE_C11702.html -> https://www.lcsc.com/product-detail/Chip-Resistor-Surface-Mount_UNI-ROYAL-Uniroyal-Elec-0402WGF2001TCE_C4109.html; Distributor Part Number C11702 -> C4109; Manufacturer Part Number 0402WGF1001TCE -> 0402WGF2001TCE; Part Description Resistor 62.5mW ±1% 1kΩ -> Resistor 62.5mW ±1% 2kΩ
- renumbered C12 to C17, C27 to C18, C28 to C19, C28 to C20, R17 to R10, R17 to R11, R23 to R13, TP3 to TP8, U6 to U2, U7 to U3
Other:
- note added: "Charge Rate: 500mA"
- note removed: "Charge Rate: 1000mA"
