File: hardware/kicad/battery.kicad_sch (KiCad schematic)
At the start: 5 parts, among them J2 +LIPO, J3 -LIPO, Q1 AO3407A

Commit message: fix schematic info
Other:
- company: (none) -> Teapot Laboratories
- title: (none) -> Battery
Changed lines of the file:
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@@
   (paper "A5")
   (title_block
-    (date "2023-10-16")
-    (rev "2")
+    (title "Battery")
+    (date "2024-01-10")
+    (rev "3")
+    (company "Teapot Laboratories")
   )
   (junction (at 106.68 52.07) (diameter 0) (color 0 0 0 0)

Commit message: update bom
Parts:
- renumbered Q1 to Q6, TP1 to TP6
Changed lines of the file:
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@@
   (symbol (lib_id "Device:Q_PMOS_GSD") (at 135.255 54.61 90) (unit 1)
     (in_bom yes) (on_board yes) (dnp no) (fields_autoplaced)
-    (property "Reference" "Q1" (at 135.255 44.45 90)
+    (property "Reference" "Q6" (at 135.255 44.45 90)
       (effects (font (size 1.27 1.27)))
     )
@@
     (instances
       (project "plantpal"
-        (path "/59b4123e-c7be-466b-a5db-658b8f0c1171"
-          (reference "Q1") (unit 1)
-        )
         (path "/59b4123e-c7be-466b-a5db-658b8f0c1171/76cc1a03-b597-4ef0-85b8-85a2d617e76b"
           (reference "Q6") (unit 1)
@@
   (symbol (lib_id "Connector:TestPoint") (at 106.68 52.07 0) (unit 1)
     (in_bom yes) (on_board yes) (dnp no)
-    (property "Reference" "TP1" (at 109.22 45.72 0)
+    (property "Reference" "TP6" (at 109.22 45.72 0)
       (effects (font (size 1.27 1.27)))
     )
@@
     (instances
       (project "plantpal"
-        (path "/59b4123e-c7be-466b-a5db-658b8f0c1171"
-          (reference "TP1") (unit 1)
-        )
         (path "/59b4123e-c7be-466b-a5db-658b8f0c1171/76cc1a03-b597-4ef0-85b8-85a2d617e76b"
           (reference "TP6") (unit 1)
@@
   (symbol (lib_id "power:+BATT") (at 149.86 48.26 0) (unit 1)
     (in_bom yes) (on_board yes) (dnp no)
-    (property "Reference" "#PWR070" (at 149.86 52.07 0)
+    (property "Reference" "#PWR091" (at 149.86 52.07 0)
       (effects (font (size 1.27 1.27)) hide)
     )
@@
     (instances
       (project "plantpal"
-        (path "/59b4123e-c7be-466b-a5db-658b8f0c1171"
-          (reference "#PWR070") (unit 1)
-        )
-        (path "/59b4123e-c7be-466b-a5db-658b8f0c1171/7fda2409-1758-4461-822b-801ba75fe202"
-          (reference "#PWR050") (unit 1)
-        )
         (path "/59b4123e-c7be-466b-a5db-658b8f0c1171/76cc1a03-b597-4ef0-85b8-85a2d617e76b"
           (reference "#PWR091") (unit 1)
@@
   (symbol (lib_id "power:+BATT") (at 69.85 44.45 0) (unit 1)
     (in_bom yes) (on_board yes) (dnp no)
-    (property "Reference" "#PWR070" (at 69.85 48.26 0)
+    (property "Reference" "#PWR089" (at 69.85 48.26 0)
       (effects (font (size 1.27 1.27)) hide)
     )
@@
     (instances
       (project "plantpal"
-        (path "/59b4123e-c7be-466b-a5db-658b8f0c1171"
-          (reference "#PWR070") (unit 1)
-        )
-        (path "/59b4123e-c7be-466b-a5db-658b8f0c1171/7fda2409-1758-4461-822b-801ba75fe202"
-          (reference "#PWR050") (unit 1)
-        )
-        (path "/59b4123e-c7be-466b-a5db-658b8f0c1171/8a163738-8cdd-43d1-ab87-ebdfd2811ec1"
-          (reference "#PWR083") (unit 1)
-        )
         (path "/59b4123e-c7be-466b-a5db-658b8f0c1171/76cc1a03-b597-4ef0-85b8-85a2d617e76b"
           (reference "#PWR089") (unit 1)
@@
   (symbol (lib_id "power:GND") (at 106.68 71.12 0) (unit 1)
     (in_bom yes) (on_board yes) (dnp no)
-    (property "Reference" "#PWR06" (at 106.68 77.47 0)
+    (property "Reference" "#PWR090" (at 106.68 77.47 0)
       (effects (font (size 1.27 1.27)) hide)
     )
@@
     (instances
       (project "plantpal"
-        (path "/59b4123e-c7be-466b-a5db-658b8f0c1171"
-          (reference "#PWR06") (unit 1)
-        )
         (path "/59b4123e-c7be-466b-a5db-658b8f0c1171/76cc1a03-b597-4ef0-85b8-85a2d617e76b"
           (reference "#PWR090") (unit 1)
