File: hardware/kicad/display.kicad_sch (KiCad schematic)
At the start: 19 parts, among them J4 HC-FPC-05-09-24RLTAG, Q7 SI1308EDL

Commit message: update bom
Parts:
- renumbered R17 to R25, R17 to R26
Changed lines of the file:
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@@
   (symbol (lib_id "Device:R_Small") (at 146.05 73.025 180) (unit 1)
     (in_bom yes) (on_board yes) (dnp no)
-    (property "Reference" "R17" (at 142.24 71.755 0)
+    (property "Reference" "R25" (at 142.24 71.755 0)
       (effects (font (size 1.27 1.27)))
     )
@@
     (instances
       (project "plantpal"
-        (path "/59b4123e-c7be-466b-a5db-658b8f0c1171"
-          (reference "R17") (unit 1)
-        )
-        (path "/59b4123e-c7be-466b-a5db-658b8f0c1171/7fda2409-1758-4461-822b-801ba75fe202"
-          (reference "R10") (unit 1)
-        )
         (path "/59b4123e-c7be-466b-a5db-658b8f0c1171/3265fc00-478b-4188-a908-4fc9b1aaf6ab"
           (reference "R25") (unit 1)
@@
   (symbol (lib_id "Device:R_Small") (at 156.21 73.025 0) (mirror x) (unit 1)
     (in_bom yes) (on_board yes) (dnp no)
-    (property "Reference" "R17" (at 160.02 71.755 0)
+    (property "Reference" "R26" (at 160.02 71.755 0)
       (effects (font (size 1.27 1.27)))
     )
@@
     (instances
       (project "plantpal"
-        (path "/59b4123e-c7be-466b-a5db-658b8f0c1171"
-          (reference "R17") (unit 1)
-        )
-        (path "/59b4123e-c7be-466b-a5db-658b8f0c1171/7fda2409-1758-4461-822b-801ba75fe202"
-          (reference "R10") (unit 1)
-        )
         (path "/59b4123e-c7be-466b-a5db-658b8f0c1171/3265fc00-478b-4188-a908-4fc9b1aaf6ab"
           (reference "R26") (unit 1)
